File: SIMAs.kicad_pcb (KiCad board)
At the start: 2 copper layers, 67.5 x 75.5 mm, 89 parts, among them J1 USB_C_Receptacle_PowerOnly_6P, J10 Conn_01x02_Pin, J11 Conn_01x03_Pin, J12 Conn_01x03_Pin, J13 Conn_01x05_Pin, J14 Conn_01x02_Pin, J2 Conn_01x02_Socket, J3 Conn_01x04_Socket, J4 Conn_01x04_Socket, J5 Conn_01x04_Socket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

Commit message: S'ha actualitzat la pcb amb els nous valors
S'ha incorporat a la pcb els canvis anteriors a l'esquemàtic, i s'ha regenerat l'ibom.
Parts:
- C20: value 100 u -> 22 u
- C7: value 20 u -> 22 u
- D4: value D -> M7
- D5, D6, D7: value 5 V -> DESD5V0S1BA-7
- D8: value 3,3 V -> SD03C-7
- D9: value 12 V -> SD12-7
- J7: value Bateria -> XT-30 male
- R14, R23: value R -> 380 k
- R21, R26: value R -> 10 k
- R22, R27: value R -> 2,5 k
- R24, R25: value R -> 100 k
