File: SIMAs.kicad_sch (KiCad schematic)
At the start: 18 parts, among them J10 Conn_01x02_Pin, J11 Conn_01x03_Pin, J12 Conn_01x03_Pin, J13 Conn_01x05_Pin, J3 Conn_01x04_Socket, J4 Conn_01x04_Socket, J5 Conn_01x04_Socket, J6 Conn_01x03_Socket, J9 Conn_01x03_Socket, U1 mini_esp32

Commit message: Nou esquemàtic
Nou esquemàtic per bateria en sèrie de dues cèl·les, boost de 12 V extern, i buck de 5 V.
Parts:
- removed J10: Conn_01x02_Pin, Connector_JST:JST_PH_B2B-PH-K_1x02_P2.00mm_Vertical, symbol Connector:Conn_01x02_Pin
Connections:
- net SENSE_ALM: now reaches U1.5 (IO_39/SVN)
Other:
- note removed: "EMERGENCY BUTTON NC"
Changed lines of the file:
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@@
 	(wire
 		(pts
-			(xy 240.03 125.73) (xy 242.57 125.73)
-		)
-		(stroke
-			(width 0)
-			(type default)
-		)
-	)
-	(wire
-		(pts
 			(xy 80.01 167.64) (xy 83.82 167.64)
 		)
@@
 	(wire
 		(pts
-			(xy 80.01 142.24) (xy 83.82 142.24)
+			(xy 82.55 152.4) (xy 83.82 152.4)
 		)
 		(stroke
@@
 	(wire
 		(pts
-			(xy 189.23 81.28) (xy 185.42 81.28)
+			(xy 80.01 142.24) (xy 83.82 142.24)
 		)
 		(stroke
@@
 	(wire
 		(pts
-			(xy 50.8 132.08) (xy 68.58 132.08)
+			(xy 189.23 81.28) (xy 185.42 81.28)
 		)
 		(stroke
@@
 	(wire
 		(pts
-			(xy 68.58 93.98) (xy 68.58 132.08)
+			(xy 50.8 132.08) (xy 68.58 132.08)
 		)
 		(stroke
@@
 	(wire
 		(pts
-			(xy 85.09 80.01) (xy 93.98 80.01)
+			(xy 68.58 93.98) (xy 68.58 132.08)
 		)
 		(stroke
@@
 	(wire
 		(pts
-			(xy 240.03 123.19) (xy 242.57 123.19)
+			(xy 85.09 80.01) (xy 93.98 80.01)
 		)
 		(stroke
@@
 		)
 	)
-	(text "EMERGENCY BUTTON NC"
-		(exclude_from_sim no)
-		(at 253.238 118.618 0)
-		(effects
-			(font
-				(size 1.27 1.27)
-			)
-		)
-	)
 	(text "GPIO"
 		(exclude_from_sim no)
@@
 		)
 	)
-	(label "VSys"
-		(at 240.03 123.19 180)
-		(effects
-			(font
-				(size 1.27 1.27)
-			)
-			(justify right bottom)
-		)
-	)
 	(label "SONS1"
 		(at 184.15 121.92 180)
@@
 		)
 	)
-	(global_label "EM_BTN"
-		(shape output)
-		(at 240.03 125.73 180)
+	(global_label "SENSE_ALM"
+		(shape input)
+		(at 82.55 152.4 180)
 		(fields_autoplaced yes)
 		(effects
@@
 		)
 		(property "Intersheetrefs" "${INTERSHEET_REFS}"
-			(at 229.9087 125.73 0)
+			(at 68.9816 152.4 0)
 			(effects
 				(font
@@
 					(unit 1)
 				)
-			)
-		)
-	)
-	(symbol
-		(lib_id "Connector:Conn_01x02_Pin")
-		(at 247.65 125.73 180)
-		(unit 1)
-		(exclude_from_sim no)
-		(in_bom yes)
-		(on_board yes)
-		(dnp no)
-		(fields_autoplaced yes)
-		(property "Reference" "J10"
-			(at 248.92 123.1899 0)
-			(effects
-				(font
-					(size 1.27 1.27)
-				)
-				(justify right)
-			)
-		)
-		(property "Value" "Conn_01x02_Pin"
-			(at 248.92 125.7299 0)
-			(effects
-				(font
-					(size 1.27 1.27)
-				)
-				(justify right)
-			)
-		)
-		(property "Footprint" "Connector_JST:JST_PH_B2B-PH-K_1x02_P2.00mm_Vertical"
-			(at 247.65 125.73 0)
-			(effects
-				(font
-					(size 1.27 1.27)
-				)
-				(hide yes)
-			)
-		)
-		(property "Datasheet" "~"
-			(at 247.65 125.73 0)
-			(effects
-				(font
-					(size 1.27 1.27)
-				)
-				(hide yes)
-			)
-		)
-		(property "Description" "Generic connector, single row, 01x02, script generated"
-			(at 247.65 125.73 0)
-			(effects
-				(font
-					(size 1.27 1.27)
-				)
-				(hide yes)
-			)
-		)
-		(pin "1"
-		)
-		(pin "2"
-		)
-		(instances
-			(project ""
-				(path "/0e086368-df4c-4139-a634-f31f7cd00dd9"
-					(reference "J10")
-					(unit 1)
-				)
